File: Hardware/main/main.kicad_sch (KiCad schematic)
At the start: 0 parts

Commit message: Rj-45 eklendi
Rj-45 eklendi linkler düzeltildi
Parts:
- added L1: ~, symbol User_HB_Library_001:inductor_User_HB
Changed lines of the file:
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@@
 		(date "2025-04-05")
+	)
+	(rule_area
+		(polyline
+			(pts
+				(xy 25.4 30.48) (xy 40.64 30.48) (xy 40.64 44.45) (xy 26.67 44.45) (xy 25.4 43.18)
+			)
+			(stroke
+				(width 0)
+				(type dash)
+			)
+			(fill
+				(type none)
+			)
+		)
+	)
+	(symbol
+		(lib_id "User_HB_Library_001:inductor_User_HB")
+		(at 31.75 39.37 0)
+		(unit 1)
+		(exclude_from_sim no)
+		(in_bom yes)
+		(on_board yes)
+		(dnp no)
+		(fields_autoplaced yes)
+		(property "Reference" "L1"
+			(at 31.75 34.29 0)
+			(effects
+				(font
+					(size 1.27 1.27)
+				)
+			)
+		)
+		(property "Value" "~"
+			(at 31.75 35.56 0)
+			(effects
+				(font
+					(size 1.27 1.27)
+				)
+			)
+		)
+		(property "Footprint" ""
+			(at 31.75 39.37 0)
+			(effects
+				(font
+					(size 1.27 1.27)
+				)
+				(hide yes)
+			)
+		)
+		(property "Datasheet" ""
+			(at 31.75 39.37 0)
+			(effects
+				(font
+					(size 1.27 1.27)
+				)
+				(hide yes)
+			)
+		)
+		(property "Description" ""
+			(at 31.75 39.37 0)
+			(effects
+				(font
+					(size 1.27 1.27)
+				)
+				(hide yes)
+			)
+		)
+		(pin "1"
+		)
+		(pin "2"
+		)
+		(instances
+			(project ""
+				(path "/a940b775-bf67-4224-b5c3-1d071abb9d1b"
+					(reference "L1")
+					(unit 1)
+				)
+			)
+		)
 	)
 	(sheet_instances
