File: Hardware/main/ETS_GIT_ETHERNET.kicad_sch (KiCad schematic)
At the start: 2 parts, among them J3 RJ45_Hanrun_HR911105A_Horizon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

Commit message: Ethernet Çizimi
Ethernet Çizimi devam ediyor  teyit lazım
Parts:
- removed J3: RJ45_Hanrun_HR911105A_Horizontal, Connector_RJ:RJ45_Hanrun_HR911105A_Horizontal, symbol Connector:RJ45_Hanrun_HR911105A_Horizontal
- added C21, C23, C24, C25, C26, C27, C28, C30, C31, C32, C34: 100nF, Capacitor_SMD:C_0805_2012Metric_Pad1.18x1.45mm_HandSolder, symbol Device:C_Small
- added C29, C33: 10nF, Capacitor_SMD:C_0805_2012Metric_Pad1.18x1.45mm_HandSolder, symbol Device:C_Small
- added J4: RJ45_Hanrun_HR911105A_Horizontal, Connector_RJ:RJ45_Hanrun_HR911105A_Horizontal, symbol Connector:RJ45_Hanrun_HR911105A_Horizontal
- added R10, R11, R8, R9: 51R, Resistor_SMD:R_0805_2012Metric_Pad1.20x1.40mm_HandSolder, symbol Device:R_Small_US
- added R12, R13: 2K, Resistor_SMD:R_0805_2012Metric_Pad1.20x1.40mm_HandSolder, symbol Device:R_Small_US
- added R14, R17: 4.7K, Resistor_SMD:R_0805_2012Metric_Pad1.20x1.40mm_HandSolder, symbol Device:R_Small_US
- added R15: 150R, Resistor_SMD:R_0805_2012Metric_Pad1.20x1.40mm_HandSolder, symbol Device:R_Small_US
- added R16: 18R, Resistor_SMD:R_0805_2012Metric_Pad1.20x1.40mm_HandSolder, symbol Device:R_Small_US
- added Y3: DFA-S15, Oscillator:Oscillator_SMD_Fordahl_DFAS15-4Pin_5.0x3.2mm, symbol Oscillator:DFA-S15
Connections:
- net RD-: now reaches U4.13 (RD-)
- net RD-: now also J4.6 (RD-), R9.2
- net RD+: now reaches U4.14 (RD+)
- net RD+: now also J4.3 (RD+), R8.1
- net GND: now reaches U4.15 (AGND_1)
- net GND: now also U4.19 (AGND_2), C21.2, C23.2, C24.2, C25.2, C26.2, C27.2, C28.2, C29.2, C30.2, C31.2, C32.2, C33.2, C34.2, J4.SH, R16.1
- net TD-: now reaches U4.16 (TD-)
- net TD-: now also J4.2 (TD-), R11.2
- net TD+: now reaches U4.17 (TD+)
- net TD+: now also J4.1 (TD+), R10.1
- net PFB: now reaches U4.18 (PFBIN1)
- net PFB: now also U4.23 (PFBOUT), C26.1, C27.1, C28.1, C29.1
- net TX_EN: now reaches U4.2 (TX_EN)
- net at U4.20 (RESERVED_1): now also R13.1
- net at U4.21 (RESERVED_2): now also R12.2
- net 3V3: now reaches U4.22 (AVDD33)
- net 3V3: now also U4.32 (IOVDD33_1), C21.1, C23.1, C24.1, C25.1, C30.1, C31.1, C32.1, C33.1, J4.12, J4.4 (TCT), J4.5 (RCT), J4.9, R10.2, R11.1, R12.1, R13.2, R8.2, R9.1
- net at U4.24 (RBIAS): now also R14.2
- net LEADCT_LINK: now reaches U4.26 (LED_ACT/COL/AN_EN)
- net LEADCT_LINK: now also J4.11
- net LED_LINK: now reaches U4.28 (LED_LINK/AN0)
- net LED_LINK: now also J4.10
- net NRST: now reaches U4.29 (RESET_N)
- net TXD0: now reaches U4.3 (TXD_0)
- net MDIO: now reaches U4.30 (MDIO)
- net MDC: now reaches U4.31 (MDC)
- net OSC1: now reaches U4.34 (X1)
- net OSC1: now also R17.1
- net TXD1: now reaches U4.4 (TXD_1)
- new net: R15.1, R16.2
- new net: R14.1, R15.2
- new net: R17.2, Y3.3 (OUT)
- new net: C34.1, J4.8

Commit message: ethernet schematik bitti
ethernet schematik bitti
Parts:
- removed J4: RJ45_Hanrun_HR911105A_Horizontal, Connector_RJ:RJ45_Hanrun_HR911105A_Horizontal, symbol Connector:RJ45_Hanrun_HR911105A_Horizontal
- removed U4: ~, User_HB_Footprints:DP83848IVVXNOPB_HB, symbol User_HB_Library:DP83848IVVXNOPB_HB
- added J5: RJ45_Wuerth_7499010211A, Connector_RJ:RJ45_Wuerth_7499010211A_Horizontal, symbol Connector:RJ45_Wuerth_7499010211A
- added R18, R19: 4.7K, Resistor_SMD:R_0805_2012Metric_Pad1.20x1.40mm_HandSolder, symbol Device:R_Small_US
- added U3: ~, User_HB_Footprints:DP83848IVVXNOPB_HB, symbol User_HB_Library:DP83848IVVXNOPB_HB
- R17: value 4.7K -> 0R
Connections:
- net 3V3: now also Y3.4 (V+), J5.12, J5.4 (CTD), J5.5 (CRD), J5.9, R18.2, R19.2, U3.22 (AVDD33), U3.32 (IOVDD33_1), U3.48 (IOVDD33_2)
- net GND: now also Y3.2 (GND), J5.SH, U3.15 (AGND_1), U3.19 (AGND_2), U3.35 (IOGND_1), U3.36 (DGND), U3.47 (IOGND_2)
- net LEADCT_LINK: now also J5.11, U3.26 (LED_ACT/COL/AN_EN)
- net LED_LINK: now also J5.10, U3.28 (LED_LINK/AN0)
- net MDC: now also U3.31 (MDC)
- net MDIO: now also U3.30 (MDIO)
- net NRST: now also U3.29 (RESET_N)
- net PFB: now also U3.18 (PFBIN1), U3.23 (PFBOUT), U3.37 (PFBIN2)
- net RD+: now also J5.3 (RD+), U3.14 (RD+)
- net RD-: now also J5.6 (RD-), U3.13 (RD-)
- net TD+: now also J5.1 (TD+), U3.17 (TD+)
- net TD-: now also J5.2 (TD-), U3.16 (TD-)
- net TXD0: now also U3.3 (TXD_0)
- net TXD1: now also U3.4 (TXD_1)
- net TX_EN: now also U3.2 (TX_EN)
- net at C34.1: now also J5.8
- net at R13.1: now also U3.20 (RESERVED_1)
- net at R12.2: now also U3.21 (RESERVED_2)
- net at R14.2: now also U3.24 (RBIAS)
- net OSC1 renamed OSCIN
- net OSCIN: now also U3.34 (X1)
- new net: R18.1, U3.39 (RX_DV/MII_MODE)
- new net CRS_DV: R19.1, U3.40 (CRS/CRS_DV/LED_CFG)
- new net RDX0: U3.43 (RXD_0/PHYAD1)
- new net RDX1: U3.44 (RXD_1/PHYAD2)
Other:
- moved on the sheet: C21, C23, C24, C25, C26, C27, C28, C29, C30, C31, C32, C33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
